Commit message: Update 3link.urdf

File: 3link.urdf (robot description, URDF)
Before this commit: robot robot_arm, 3 links, 2 joints
Joints:
- removed joint joint_1
- removed joint joint_2
- added joint joint1: type continuous, parent link1, child link2, origin xyz=0 .1 0 rpy=0 0 0, axis 0 0 1, limit lower=-3.141592653589793 upper=3.141592653589793 effort=1000.0 velocity=2.5
- added joint joint2: type continuous, parent link2, child link3, origin xyz=0.3536 0.3536 0.25 rpy=0 0 0, axis 0 0 1, limit lower=-3.141592653589793 upper=3.141592653589793 effort=1000.0 velocity=2.5
