Commit message: Update 3link (1).urdf

File: 3link (1).urdf (robot description, URDF)
Before this commit: robot robot_arm, 3 links, 2 joints
Joints:
- joint joint2: type fixed -> continious

Commit message: Update 3link (1).urdf

File: 3link (1).urdf (robot description, URDF)
Before this commit: robot robot_arm, 3 links, 2 joints
Joints:
- joint joint1: origin xyz=0 0 0 rpy=0 0 0 -> xyz=0 0 .1 rpy=0 0 0

Commit message: Update 3link (1).urdf

File: 3link (1).urdf (robot description, URDF)
Before this commit: robot robot_arm, 3 links, 2 joints
Joints:
- joint joint2: origin xyz=0 0 0 rpy=0 0 0 -> xyz=0 0 .7 rpy=0 0 0

Commit message: Update 3link (1).urdf

File: 3link (1).urdf (robot description, URDF)
Before this commit: robot robot_arm, 3 links, 2 joints
Joints:
- joint joint2: type continious -> fixed

Commit message: Update 3link (1).urdf

File: 3link (1).urdf (robot description, URDF)
Before this commit: robot robot_arm, 3 links, 2 joints
Joints:
- joint joint1: origin xyz=0 0 .1 rpy=0 0 0 -> xyz=0 .1 .3 rpy=0 0 0
- joint joint2: origin xyz=0 0 .7 rpy=0 0 0 -> xyz=0 .2 .7 rpy=0 0 0

Commit message: Update 3link (1).urdf

File: 3link (1).urdf (robot description, URDF)
Before this commit: robot robot_arm, 3 links, 2 joints
Joints:
- joint joint2: origin xyz=0 .2 .7 rpy=0 0 0 -> xyz=0 .2 .6 rpy=0 0 0

Commit message: Update 3link (1).urdf

File: 3link (1).urdf (robot description, URDF)
Before this commit: robot robot_arm, 3 links, 2 joints
Joints:
- joint joint2: origin xyz=0 .2 .6 rpy=0 0 0 -> xyz=0 .1 .5 rpy=0 0 0

Commit message: Update 3link (1).urdf

File: 3link (1).urdf (robot description, URDF)
Before this commit: robot robot_arm, 3 links, 2 joints
Joints:
- joint joint2: origin xyz=0 .1 .5 rpy=0 0 0 -> xyz=0 .1 .3 rpy=0 0 0

Commit message: Update 3link (1).urdf

File: 3link (1).urdf (robot description, URDF)
Before this commit: robot robot_arm, 3 links, 2 joints
Joints:
- joint joint1: origin xyz=0 .1 .3 rpy=0 0 0 -> xyz=0 0 .1 rpy=0 0 0

Commit message: Update 3link (1).urdf

File: 3link (1).urdf (robot description, URDF)
Before this commit: robot robot_arm, 3 links, 2 joints
Joints:
- joint joint1: origin xyz=0 0 .1 rpy=0 0 0 -> xyz=0 .1 .3 rpy=0 0 0

Commit message: Update 3link (1).urdf

File: 3link (1).urdf (robot description, URDF)
Before this commit: robot robot_arm, 3 links, 2 joints
Joints:
- joint joint1: type fixed -> revolute
- joint joint2: type fixed -> revolute

Commit message: Update 3link (1).urdf

File: 3link (1).urdf (robot description, URDF)
Before this commit: robot robot_arm, 3 links, 2 joints
Joints:
- joint joint1: axis 0 0 0 -> 0 0 1
- joint joint2: axis (none) -> 0 0 1; limit (none) -> lower=-3.141592653589793 upper=3.141592653589793 effort=1000.0 velocity=2.5

Commit message: Update 3link (1).urdf

File: 3link (1).urdf (robot description, URDF)
Before this commit: robot robot_arm, 3 links, 2 joints
Joints:
- joint joint1: axis 0 0 1 -> 1 0 0
- joint joint2: axis 0 0 1 -> 1 0 0

Commit message: Update 3link (1).urdf

File: 3link (1).urdf (robot description, URDF)
Before this commit: robot robot_arm, 3 links, 2 joints
Joints:
- joint joint1: axis 1 0 0 -> 0 1 0
- joint joint2: axis 1 0 0 -> 0 1 0
