Commit message: Update 3link1.urdf

File: 3link1.urdf (robot description, URDF)
Before this commit: robot three_link_robot, 3 links, 2 joints
Links:
- link link1: geometry collision box size=.1 .2 .1; visual box size=.1 .2 .1
- link link2: geometry collision cylinder length=0.5 radius=0.1; visual cylinder length=0.5 radius=0.1
- link link3: geometry collision cylinder length=0.5 radius=0.1; visual cylinder length=0.5 radius=0.1
Joints:
- joint joint1: axis (none) -> 0 0 1; limit (none) -> lower=-3.141592653589793 upper=3.141592653589793 effort=1000.0 velocity=2.5; origin xyz=0 0.1 0 rpy=0 0 0 -> xyz=0 .1 .3 rpy=0 0 0; type fixed -> revolute
- joint joint2: axis (none) -> 0 1 0; limit (none) -> lower=-3.141592653589793 upper=3.141592653589793 effort=1000.0 velocity=2.5; origin xyz=0.3536 0.3536 0.25 rpy=0 0 0 -> xyz=0 .2 .25 rpy=0 0 0; type fixed -> revolute

Commit message: Update 3link1.urdf

File: 3link1.urdf (robot description, URDF)
Before this commit: robot robot_arm, 3 links, 2 joints
Joints:
- joint joint2: origin xyz=0 .2 .25 rpy=0 0 0 -> xyz=0 .15 .25 rpy=0 0 0

Commit message: Update 3link1.urdf

File: 3link1.urdf (robot description, URDF)
Before this commit: robot robot_arm, 3 links, 2 joints
Joints:
- joint joint1: origin xyz=0 .1 .3 rpy=0 0 0 -> xyz=0 .15 0 rpy=0 0 0

Commit message: Update 3link1.urdf

File: 3link1.urdf (robot description, URDF)
Before this commit: robot robot_arm, 3 links, 2 joints
Joints:
- joint joint1: origin xyz=0 .15 0 rpy=0 0 0 -> xyz=0 0 0 rpy=0 0 0
- joint joint2: origin xyz=0 .15 .25 rpy=0 0 0 -> xyz=0 .15 .35 rpy=0 0 0

Commit message: Update 3link1.urdf

File: 3link1.urdf (robot description, URDF)
Before this commit: robot robot_arm, 3 links, 2 joints
Joints:
- joint joint2: origin xyz=0 .15 .35 rpy=0 0 0 -> xyz=0 .15 .5 rpy=0 0 0

Commit message: Update 3link1.urdf

File: 3link1.urdf (robot description, URDF)
Before this commit: robot robot_arm, 3 links, 2 joints
Joints:
- joint joint1: origin xyz=0 0 .1 rpy=0 0 0 -> xyz=0 0 .5 rpy=0 0 0

Commit message: Update 3link1.urdf

File: 3link1.urdf (robot description, URDF)
Before this commit: robot robot_arm, 3 links, 2 joints
Joints:
- joint joint1: origin xyz=0 0 .5 rpy=0 0 0 -> xyz=0 0 .05 rpy=0 0 0

Commit message: Update 3link1.urdf

File: 3link1.urdf (robot description, URDF)
Before this commit: robot robot_arm, 3 links, 2 joints
Joints:
- joint joint2: origin xyz=0 .15 .5 rpy=0 0 0 -> xyz=0 .2 .5 rpy=0 0 0

Commit message: Update 3link1.urdf

File: 3link1.urdf (robot description, URDF)
Before this commit: robot robot_arm, 3 links, 2 joints
Joints:
- joint joint1: axis 0 0 1 -> 0 1 0
